Commit message: feat: align upstream sources and bilingual tutorials

File: ros2_ws/src/microduck_description/urdf/microduck.urdf.xacro (robot description, xacro)
@@ -1,5 +1,5 @@
 <?xml version='1.0' encoding='utf-8'?>
 <robot name="microduck" xmlns:xacro="http://www.ros.org/wiki/xacro">
-  <!-- Generated from Pollen Robotics microduck_rl robot_allcollisions.xml at d424a0c899f6b33cbd3daeb279913134349c0b63. Do not hand-edit generated geometry. -->
+  <!-- Generated from Pollen Robotics microduck_rl robot_groundcontact.xml at ceca01706143d729305baa94cbd8ab990979e325. Do not hand-edit generated geometry. -->
   <xacro:arg name="with_visual_meshes" default="true" />
   <xacro:arg name="with_collision_meshes" default="true" />
@@ -7,8 +7,8 @@
   <!-- joint_velocity_limit is a documented simulation/planning fallback; the upstream MJCF does not provide authoritative per-joint velocity limits. -->
   <material name="ankle_left_material">
-    <color rgba="0.980392 0.713725 0.00392157 1" />
+    <color rgba="1 0.403922 0.121569 1" />
   </material>
   <material name="ankle_right_material">
-    <color rgba="0.980392 0.713725 0.00392157 1" />
+    <color rgba="1 0.403922 0.121569 1" />
   </material>
   <material name="banana_pcb_locker_material">
@@ -16,8 +16,8 @@
   </material>
   <material name="bearing_roll_material">
-    <color rgba="0.262745 0.282353 0.301961 1" />
+    <color rgba="0.129412 0.152941 0.129412 1" />
   </material>
   <material name="bottom_head_shell_material">
-    <color rgba="0.980392 0.713725 0.00392157 1" />
+    <color rgba="1 0.403922 0.121569 1" />
   </material>
   <material name="elec_rpi_robot_hat_pcb_material">
@@ -25,17 +25,17 @@
   </material>
   <material name="face_part_material">
-    <color rgba="0.34902 0.376471 0.4 1" />
+    <color rgba="0.67451 0.639216 0.603922 1" />
   </material>
   <material name="foot_left_material">
-    <color rgba="0.980392 0.713725 0.00392157 1" />
+    <color rgba="1 0.403922 0.121569 1" />
   </material>
   <material name="foot_right_material">
-    <color rgba="0.980392 0.713725 0.00392157 1" />
+    <color rgba="1 0.403922 0.121569 1" />
   </material>
   <material name="hip_l_material">
-    <color rgba="0.901961 0.901961 0.901961 1" />
+    <color rgba="0.67451 0.639216 0.603922 1" />
   </material>
   <material name="jaw_material">
-    <color rgba="0.980392 0.713725 0.00392157 1" />
+    <color rgba="1 0.403922 0.121569 1" />
   </material>
   <material name="jaw_soft_material">
@@ -46,5 +46,5 @@
   </material>
   <material name="leg_material">
-    <color rgba="0.811765 0.858824 0.898039 1" />
+    <color rgba="0.67451 0.639216 0.603922 1" />
   </material>
   <material name="lens_material">
@@ -55,8 +55,8 @@
   </material>
   <material name="motor_support_material">
-    <color rgba="0.262745 0.282353 0.301961 1" />
+    <color rgba="0.129412 0.152941 0.129412 1" />
   </material>
   <material name="neck_material">
-    <color rgba="0.8 0.8 0.8 1" />
+    <color rgba="0.67451 0.639216 0.603922 1" />
   </material>
   <material name="neck_pitch_material">
@@ -64,8 +64,8 @@
   </material>
   <material name="noenoeil_material">
-    <color rgba="0.262745 0.282353 0.301961 1" />
+    <color rgba="0.956863 0.686275 0.137255 1" />
   </material>
   <material name="np_f970_material">
-    <color rgba="0.901961 0.901961 0.901961 1" />
+    <color rgba="0.301961 0.301961 0.301961 1" />
   </material>
   <material name="pcb__raspberry_pi_zero_2_w_material">
@@ -73,14 +73,14 @@
   </material>
   <material name="power_support_material">
-    <color rgba="0.901961 0.901961 0.901961 1" />
+    <color rgba="0.67451 0.639216 0.603922 1" />
   </material>
   <material name="right_shell_material">
-    <color rgba="0.8 0.8 0.8 1" />
+    <color rgba="0.85098 0.85098 0.839216 1" />
   </material>
   <material name="seeed_bearing__configuration__22x16x4_material">
-    <color rgba="0.713725 0.760784 0.8 1" />
+    <color rgba="0.811765 0.858824 0.898039 1" />
   </material>
   <material name="seeed_bearing__configuration_default_material">
-    <color rgba="0.713725 0.760784 0.8 1" />
+    <color rgba="0.811765 0.858824 0.898039 1" />
   </material>
   <material name="soft_mouth_top_material">
@@ -88,8 +88,8 @@
   </material>
   <material name="sole_left_material">
-    <color rgba="0.537255 0.854902 0.827451 1" />
+    <color rgba="0.956863 0.686275 0.137255 1" />
   </material>
   <material name="sole_right_material">
-    <color rgba="0.537255 0.854902 0.827451 1" />
+    <color rgba="0.956863 0.686275 0.137255 1" />
   </material>
   <material name="speaker_material">
@@ -97,17 +97,17 @@
   </material>
   <material name="top_head_shell_material">
-    <color rgba="0.901961 0.901961 0.901961 1" />
+    <color rgba="0.85098 0.85098 0.839216 1" />
   </material>
   <material name="trunk_base_material">
-    <color rgba="0.34902 0.376471 0.4 1" />
+    <color rgba="0.129412 0.152941 0.129412 1" />
   </material>
   <material name="upper_leg_left_material">
-    <color rgba="0.866667 0.866667 0.866667 1" />
+    <color rgba="0.85098 0.85098 0.839216 1" />
   </material>
   <material name="upper_leg_right_material">
-    <color rgba="0.866667 0.866667 0.866667 1" />
+    <color rgba="0.85098 0.85098 0.839216 1" />
   </material>
   <material name="upper_leg_rigidity_plate_material">
-    <color rgba="0.537255 0.854902 0.827451 1" />
+    <color rgba="0.67451 0.639216 0.603922 1" />
   </material>
   <material name="xl330_material">
@@ -115,8 +115,8 @@
   </material>
   <material name="yaw2roll_material">
-    <color rgba="0.647059 0.647059 0.647059 1" />
+    <color rgba="0.129412 0.152941 0.129412 1" />
   </material>
   <material name="yaw_roll_motion_material">
-    <color rgba="0.768627 0.886275 0.952941 1" />
+    <color rgba="0.129412 0.152941 0.129412 1" />
   </material>
   <link name="base_link" />
@@ -157,5 +157,5 @@
       </visual>
       <visual name="trunk_base_visual_4">
-        <origin xyz="0.006 0.0175 0.0115" rpy="3.14159265359 -1.57079632679 0" />
+        <origin xyz="0.006 0.0175 0.0115" rpy="-3.14159265359 -1.57079632679 0" />
         <geometry>
           <mesh filename="package://microduck_description/meshes/xl330.stl" />
@@ -178,5 +178,5 @@
       </visual>
       <visual name="trunk_base_visual_7">
-        <origin xyz="0.006 -0.0175 0.0115" rpy="3.14159265359 -1.57079632679 0" />
+        <origin xyz="0.006 -0.0175 0.0115" rpy="-3.14159265359 -1.57079632679 0" />
         <geometry>
           <mesh filename="package://microduck_description/meshes/xl330.stl" />
@@ -341,5 +341,5 @@
     <origin xyz="0.025 0 -0.0185" rpy="-1.57079632679 0 -1.57079632679" />
     <axis xyz="0 0 1" />
-    <limit lower="-1.5707963268" upper="1.57079632679" effort="0.96" velocity="$(arg joint_velocity_limit)" />
+    <limit lower="-1.57079632679" upper="1.57079632679" effort="0.96" velocity="$(arg joint_velocity_limit)" />
     <dynamics damping="0.053" friction="0.0048" />
   </joint>
@@ -380,12 +380,12 @@
     <origin xyz="0.022 0.0357771 -0.004" rpy="3.14159265359 0 1.57079632679" />
     <axis xyz="0 0 1" />
-    <limit lower="-1.5707963268" upper="1.57079632679" effort="0.96" velocity="$(arg joint_velocity_limit)" />
+    <limit lower="-1.57079632679" upper="1.57079632679" effort="0.96" velocity="$(arg joint_velocity_limit)" />
     <dynamics damping="0.053" friction="0.0048" />
   </joint>
   <link name="ankle_left">
     <inertial>
-      <origin xyz="-0.00615738 -0.0137483 -0.0156586" rpy="0 0 0" />
+      <origin xyz="-0.00615742 -0.0137483 -0.0156585" rpy="0 0 0" />
       <mass value="0.0300246" />
-      <inertia ixx="5.91525e-06" iyy="1.11534e-05" izz="7.74015e-06" ixy="-2.0535e-07" ixz="8.2152e-08" iyz="5.6714e-08" />
+      <inertia ixx="5.91525e-06" iyy="1.11534e-05" izz="7.74016e-06" ixy="-2.05354e-07" ixz="8.218e-08" iyz="5.6722e-08" />
     </inertial>
     <xacro:if value="$(arg with_visual_meshes)">
@@ -431,5 +431,5 @@
     <parent link="leg" />
     <child link="ankle_left" />
-    <origin xyz="0 0.042 -0.026" rpy="3.14159265359 0 0" />
+    <origin xyz="0 0.042 -0.026" rpy="-3.14159265359 0 0" />
     <axis xyz="0 0 1" />
     <limit lower="-1.57079632679" upper="1.57079632679" effort="0.96" velocity="$(arg joint_velocity_limit)" />
@@ -552,5 +552,5 @@
     <parent link="neck_pitch" />
     <child link="yaw_roll_motion" />
-    <origin xyz="0 0.0186931 -0.0145" rpy="1.57079632679 0 -3.14159265359" />
+    <origin xyz="0 0.0186931 -0.0145" rpy="1.57079632679 0 3.14159265359" />
     <axis xyz="0 0 1" />
     <limit lower="-2.96705972839" upper="2.96705972839" effort="0.96" velocity="$(arg joint_velocity_limit)" />
@@ -561,5 +561,5 @@
       <origin xyz="0.00460523 0.00120047 -0.0324761" rpy="0 0 0" />
       <mass value="0.188766" />
-      <inertia ixx="0.000320812" iyy="0.0002541" izz="0.000149882" ixy="-6.32292e-07" ixz="6.57154e-06" iyz="4.18476e-06" />
+      <inertia ixx="0.000320811" iyy="0.0002541" izz="0.000149882" ixy="-6.32293e-07" ixz="6.57153e-06" iyz="4.18477e-06" />
     </inertial>
     <xacro:if value="$(arg with_visual_meshes)">
@@ -721,5 +721,5 @@
       </visual>
       <visual name="bearing_roll_visual_1">
-        <origin xyz="0 0 0.0125" rpy="-3.14159265359 0 -1.57079632679" />
+        <origin xyz="0 0 0.0125" rpy="3.14159265359 0 -1.57079632679" />
         <geometry>
           <mesh filename="package://microduck_description/meshes/xl330.stl" />
@@ -746,5 +746,5 @@
     <parent link="trunk_base" />
     <child link="bearing_roll" />
-    <origin xyz="0.006 -0.0175 -0.005" rpy="3.14159265359 0 1.57079632679" />
+    <origin xyz="0.006 -0.0175 -0.005" rpy="-3.14159265359 0 1.57079632679" />
     <axis xyz="0 0 1" />
     <limit lower="-0.523598775598" upper="0.436332312999" effort="0.96" velocity="$(arg joint_velocity_limit)" />
@@ -885,5 +885,5 @@
       <origin xyz="0.00615539 -0.0137482 -0.0156566" rpy="0 0 0" />
       <mass value="0.0300251" />
-      <inertia ixx="5.91534e-06" iyy="1.11534e-05" izz="7.74016e-06" ixy="2.04877e-07" ixz="-8.247e-08" iyz="5.7017e-08" />
+      <inertia ixx="5.91534e-06" iyy="1.11534e-05" izz="7.74015e-06" ixy="2.04877e-07" ixz="-8.2467e-08" iyz="5.7017e-08" />
     </inertial>
     <xacro:if value="$(arg with_visual_meshes)">
